File: Rev A/PowerModule.kicad_pcb (KiCad board)
At the start: 2 copper layers, 0 parts

Commit message: Added all schematic parts, started layout
Parts:
- added C1: 1uF, Capacitor_SMD:C_0805_2012Metric, F.Cu at (139.0, 58.0)
- added C10: 1uF, Capacitor_SMD:C_0805_2012Metric, F.Cu at (130.0, 55.0)
- added C11: 1uF, Capacitor_SMD:C_0805_2012Metric, F.Cu at (112.0, 55.0)
- added C2: 10nF, Capacitor_SMD:C_0805_2012Metric, F.Cu at (151.0, 62.0)
- added C3: 1uF, Capacitor_SMD:C_0805_2012Metric, F.Cu at (131.0, 97.9)
- added C4: 1uF, Capacitor_SMD:C_0805_2012Metric, F.Cu at (131.0, 71.0)
- added C5: 10nF, Capacitor_SMD:C_0805_2012Metric, F.Cu at (151.0, 89.0)
- added C6: 100nF, Capacitor_SMD:C_0805_2012Metric, F.Cu at (151.0, 86.0)
- added C7: 100nF, Capacitor_SMD:C_0805_2012Metric, F.Cu at (151.0, 113.0)
- added C8: 1uF, Capacitor_SMD:C_0805_2012Metric, F.Cu at (112.0, 58.0)
- added C9: 1uF, Capacitor_SMD:C_0805_2012Metric, F.Cu at (130.0, 58.0)
- added D1: 1N5819W, Diode_SMD:D_SOD-123F, F.Cu at (178.0, 30.0)
- added D10: LED Blue, LED_SMD:LED_0805_2012Metric, F.Cu at (131.0, 109.9)
- added D11: LED WHITE, LED_SMD:LED_0805_2012Metric, F.Cu at (170.0, 104.0)
- added D12: SMAZ15Z-13-F, Diode_SMD:D_SMA, F.Cu at (179.0, 101.0)
- added D13: LED Yellow, LED_SMD:LED_0805_2012Metric, F.Cu at (139.0, 46.0)
- added D14: LED Orange, LED_SMD:LED_0805_2012Metric, F.Cu at (157.0, 40.0)
- added D15: LED Blue, LED_SMD:LED_0805_2012Metric, F.Cu at (157.0, 53.0)
- added D16: 1N5819W, Diode_SMD:D_SOD-123F, F.Cu at (130.0, 41.0)
- added D17: 1N5819W, Diode_SMD:D_SOD-123F, F.Cu at (112.0, 41.0)
- added D18: LED WHITE, LED_SMD:LED_0805_2012Metric, F.Cu at (112.0, 49.0)
- added D19: LED WHITE, LED_SMD:LED_0805_2012Metric, F.Cu at (130.0, 49.0)
- added D2: 1N5819W, Diode_SMD:D_SOD-123F, F.Cu at (168.0, 30.0)
- added D20: SZSMF4L15CAT3G, Diode_SMD:D_SOD-123F, F.Cu at (174.0, 74.0)
- added D21: SZSMF4L15CAT3G, Diode_SMD:D_SOD-123F, F.Cu at (174.0, 101.0)
- added D22: SMAZ15Z-13-F, Diode_SMD:D_SMA, F.Cu at (104.0, 36.0)
- added D23: SZSMF4L15CAT3G, Diode_SMD:D_SOD-123F, F.Cu at (100.0, 36.0)
- added D24: SMAZ15Z-13-F, Diode_SMD:D_SMA, F.Cu at (190.0, 36.0)
- added D25: SZSMF4L15CAT3G, Diode_SMD:D_SOD-123F, F.Cu at (194.0, 36.0)
- added D26: SMAJ5.0CA, Diode_SMD:D_SMA, F.Cu at (85.0, 69.9)
- added D27: SMAJ5.0CA, Diode_SMD:D_SMA, F.Cu at (85.0, 74.5)
- added D28: SMAJ5.0CA, Diode_SMD:D_SMA, F.Cu at (85.0, 79.0)
- added D29: SMAJ5.0CA, Diode_SMD:D_SMA, F.Cu at (85.0, 83.5)
- added D3: SMAZ15Z-13-F, Diode_SMD:D_SMA, F.Cu at (179.0, 74.0)
- added D30: SMAJ5.0CA, Diode_SMD:D_SMA, F.Cu at (85.0, 88.1)
- added D4: LED Yellow, LED_SMD:LED_0805_2012Metric, F.Cu at (123.2, 69.0)
- added D5: LED Green, LED_SMD:LED_0805_2012Metric, F.Cu at (131.0, 83.0)
- added D6: LED Orange, LED_SMD:LED_0805_2012Metric, F.Cu at (136.0, 62.0)
- added D7: LED Yellow, LED_SMD:LED_0805_2012Metric, F.Cu at (123.1, 73.0)
- added D8: LED WHITE, LED_SMD:LED_0805_2012Metric, F.Cu at (170.0, 77.0)
- added D9: LED Orange, LED_SMD:LED_0805_2012Metric, F.Cu at (136.0, 89.0)
- added H1: M3 Hole, MountingHole:MountingHole_3.2mm_M3_Pad_TopBottom, F.Cu at (192.0, 28.0)
- added H2: M3 Hole, MountingHole:MountingHole_3.2mm_M3_Pad_TopBottom, F.Cu at (102.0, 28.0)
- added H3: M3 Hole, MountingHole:MountingHole_3.2mm_M3_Pad_TopBottom, F.Cu at (192.0, 118.0)
- added H4: M3 Hole, MountingHole:MountingHole_3.2mm_M3_Pad_TopBottom, F.Cu at (102.0, 118.0)
- added J1: NC6-P108-02, TerminalBlock_MetzConnect:TerminalBlock_MetzConnect_Type703_RT10N02HGLU_1x02_P9.52mm_Horizontal, F.Cu at (191.8, 69.2)
- added J2: NC6-P108-02, TerminalBlock_MetzConnect:TerminalBlock_MetzConnect_Type703_RT10N02HGLU_1x02_P9.52mm_Horizontal, F.Cu at (191.8, 96.2)
- added J3: 1x7 Socket P2.54mm, Connector_PinSocket_2.54mm:PinSocket_1x07_P2.54mm_Vertical, B.Cu at (102.0, 65.4)
- added K1: Relay_SPDT, MosfetsRelaysSwitches_Surgical_Lighting:TE_VCF4-1000, F.Cu at (173.0, 46.0)
- added Q1: IRLZ44N, Package_TO_SOT_THT:TO-220-3_Horizontal_TabDown, F.Cu at (145.5, 58.2)
- added Q2: IRLZ44N, Package_TO_SOT_THT:TO-220-3_Horizontal_TabDown, F.Cu at (159.5, 84.2)
- added Q3: IRLZ44N, Package_TO_SOT_THT:TO-220-3_Horizontal_TabDown, F.Cu at (159.5, 111.2)
- added R1: 1K, Resistor_SMD:R_0805_2012Metric, F.Cu at (139.0, 52.0)
- added R10: 10K, Resistor_SMD:R_0805_2012Metric, F.Cu at (131.0, 77.0)
- added R11: 10K, Resistor_SMD:R_0805_2012Metric, F.Cu at (151.0, 80.0)
- added R12: 10K, Resistor_SMD:R_0805_2012Metric, F.Cu at (151.0, 77.0)
- added R13: 0805,1k, Resistor_SMD:R_0805_2012Metric, F.Cu at (119.1, 69.0)
- added R14: 10K, Resistor_SMD:R_0805_2012Metric, F.Cu at (151.1, 101.0)
- added R15: 10K, Resistor_SMD:R_0805_2012Metric, F.Cu at (151.0, 98.0)
- added R16: 0805,1k, Resistor_SMD:R_0805_2012Metric, F.Cu at (131.0, 89.0)
- added R17: 100R, Resistor_SMD:R_0805_2012Metric, F.Cu at (151.0, 95.0)
- added R18: 100K, Resistor_SMD:R_0805_2012Metric, F.Cu at (151.0, 92.0)
- added R19: 10K, Resistor_SMD:R_0805_2012Metric, F.Cu at (131.0, 92.0)
- added R2: 100K, Resistor_SMD:R_0805_2012Metric, F.Cu at (139.0, 55.0)
- added R20: 10K, Resistor_SMD:R_0805_2012Metric, F.Cu at (131.0, 101.0)
- added R21: 10K, Resistor_SMD:R_0805_2012Metric, F.Cu at (131.0, 106.9)
- added R22: 10K, Resistor_SMD:R_0805_2012Metric, F.Cu at (131.0, 94.9)
- added R23: 100R, Resistor_SMD:R_0805_2012Metric, F.Cu at (151.0, 83.0)
- added R24: 10K, Resistor_SMD:R_0805_2012Metric, F.Cu at (131.0, 103.9)
- added R25: 0805,1k, Resistor_SMD:R_0805_2012Metric, F.Cu at (131.0, 86.0)
- added R26: 10K, Resistor_SMD:R_0805_2012Metric, F.Cu at (151.0, 74.0)
- added R27: 10K, Resistor_SMD:R_0805_2012Metric, F.Cu at (151.0, 71.0)
- added R28: 0805,1k, Resistor_SMD:R_0805_2012Metric, F.Cu at (131.0, 62.0)
- added R29: 0805,1k, Resistor_SMD:R_0805_2012Metric, F.Cu at (119.0, 73.0)
- added R3: 100R, Resistor_SMD:R_0805_2012Metric, F.Cu at (151.0, 68.0)
- added R30: 0805,10k, Resistor_SMD:R_0805_2012Metric, F.Cu at (170.0, 71.0)
- added R31: 5mR 1W, Resistor_SMD:R_2512_6332Metric, F.Cu at (175.0, 109.0)
- added R32: 10K, Resistor_SMD:R_0805_2012Metric, F.Cu at (151.0, 104.0)
- added R33: 10K, Resistor_SMD:R_0805_2012Metric, F.Cu at (151.0, 107.0)
- added R34: 0805,1k, Resistor_SMD:R_0805_2012Metric, F.Cu at (131.0, 112.9)
- added R35: 0805,10k, Resistor_SMD:R_0805_2012Metric, F.Cu at (170.0, 98.0)
- added R36: 100R, Resistor_SMD:R_0805_2012Metric, F.Cu at (151.0, 110.0)
- added R37: 0805,10k, Resistor_SMD:R_0805_2012Metric, F.Cu at (157.0, 35.0)
- added R38: 0805,1k, Resistor_SMD:R_0805_2012Metric, F.Cu at (139.0, 49.0)
- added R39: 0805,10k, Resistor_SMD:R_0805_2012Metric, F.Cu at (157.0, 58.0)
- added R4: 100K, Resistor_SMD:R_0805_2012Metric, F.Cu at (151.0, 65.0)
- added R40: 0805,10k, Resistor_SMD:R_0805_2012Metric, F.Cu at (112.0, 52.0)
- added R41: 0805,1k, Resistor_SMD:R_0805_2012Metric, F.Cu at (130.0, 52.0)
- added R5: 5mR 1W, Resistor_SMD:R_2512_6332Metric, F.Cu at (175.0, 82.0)
- added R6: 10K, Resistor_SMD:R_0805_2012Metric, F.Cu at (131.0, 74.0)
- added R7: 10K, Resistor_SMD:R_0805_2012Metric, F.Cu at (131.0, 65.0)
- added R8: 10K, Resistor_SMD:R_0805_2012Metric, F.Cu at (131.0, 80.0)
- added R9: 10K, Resistor_SMD:R_0805_2012Metric, F.Cu at (131.0, 68.0)
- added TP1: TestPoint_Small, TestPoint:TestPoint_Pad_D2.0mm, F.Cu at (172.0, 87.0)
- added TP10: TestPoint_Small, TestPoint:TestPoint_Pad_D2.0mm, F.Cu at (115.0, 77.0)
- added TP2: TestPoint_Small, TestPoint:TestPoint_Pad_D2.0mm, F.Cu at (178.0, 87.0)
- added TP3: TestPoint_Small, TestPoint:TestPoint_Pad_D2.0mm, F.Cu at (115.0, 81.0)
- added TP4: TestPoint_Small, TestPoint:TestPoint_Pad_D2.0mm, F.Cu at (159.5, 87.3)
- added TP5: TestPoint_Small, TestPoint:TestPoint_Pad_D2.0mm, F.Cu at (115.0, 73.0)
- added TP6: TestPoint_Small, TestPoint:TestPoint_Pad_D2.0mm, F.Cu at (115.0, 69.0)
- added TP7: TestPoint_Small, TestPoint:TestPoint_Pad_D2.0mm, F.Cu at (172.0, 114.0)
- added TP8: TestPoint_Small, TestPoint:TestPoint_Pad_D2.0mm, F.Cu at (178.0, 114.0)
- added TP9: TestPoint_Small, TestPoint:TestPoint_Pad_D2.0mm, F.Cu at (159.4, 114.1)
- added U1: LM324, Package_DIP:DIP-14_W7.62mm_Socket, F.Cu at (137.2, 66.4)
- added U2: LM324, Package_DIP:DIP-14_W7.62mm_Socket, F.Cu at (137.2, 93.4)
- added U3: LM7805, Package_TO_SOT_THT:TO-220-3_Horizontal_TabDown, F.Cu at (118.5, 58.2)
Other:
- board outline added: 100 x 100 mm
