File: Rev A/PowerModule.kicad_pcb (KiCad board)
At the start: 2 copper layers, 100 x 100 mm, 106 parts, among them J1 NC6-P108-02, J2 NC6-P108-02, J3 1x7 Socket P2.54mm, K1 Relay_SPDT, Q1 IRLZ44N, Q2 IRLZ44N, Q3 IRLZ44N, U1 LM324, U2 LM324, U3 LM7805

Commit message: laid out pcb
Parts:
- added R42: 0805,0, Resistor_SMD:R_0805_2012Metric, F.Cu at (121.0, 52.0)
- C6, C7: value 100nF -> 10nF
- D10: value LED Blue -> LED Green
- D26, D27, D28, D29, D30: value SMAJ5.0CA -> PESD3V3L1BA,115; footprint Diode_SMD:D_SMA -> Diode_SMD:D_SOD-323F
- R23, R36: value 100R -> 1K
- moved R36 41.7 mm to (115.0, 89.0), turned to 180 degrees
- moved C7 39.2 mm to (120.0, 89.0), turned to 0 degrees
- moved R23 36.1 mm to (115.0, 85.0), turned to 180 degrees
- moved R34 35.7 mm to (115.0, 81.0)
- moved C6 31.0 mm to (120.0, 85.0), turned to 0 degrees
- moved D10 30.9 mm to (120.0, 81.0), turned to 180 degrees
- moved R38 28.8 mm to (115.0, 65.0)
- moved D13 26.9 mm to (120.0, 65.0), turned to 180 degrees
- moved D30 23.8 mm to (107.0, 79.0), turned to 180 degrees
- moved D29 23.3 mm to (107.0, 76.0), turned to 180 degrees
- moved D28 22.8 mm to (107.0, 73.0), turned to 180 degrees
- moved D27 22.4 mm to (107.0, 70.0), turned to 180 degrees
- moved D26 22.2 mm to (107.0, 67.0), turned to 180 degrees
- moved R25 18.4 mm to (115.0, 77.0)
- moved D5 12.5 mm to (120.0, 77.0), turned to 180 degrees
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Connections:
- net +5VA renamed /OpAmpPWR
- net Net-(D16-K) renamed /VIN_OPA_PWR
- net Net-(R11-Pad2) renamed /ISen1_unfilt
- net Net-(R33-Pad2) renamed /ISen2_unfilt
- C6 pad 1: /CurrentSenseCh2 -> /CurrentSenseCh1
- C7 pad 1: /CurrentSenseCh1 -> /CurrentSenseCh2
- D11 pad 1: /ISense1_P -> /ISense2_P
- D12 pad 2: /ISense1_P -> /ISense2_P
- D20 pad 1: /ISense2_P -> /ISense1_P
- D21 pad 1: /ISense1_P -> /ISense2_P
- D3 pad 2: /ISense2_P -> /ISense1_P
- D8 pad 1: /ISense2_P -> /ISense1_P
- J1 pad 2: /ISense2_P -> /ISense1_P
- J2 pad 2: /ISense1_P -> /ISense2_P
- Q2 pad 2: /ISense2_N -> /ISense1_N
- Q3 pad 2: /ISense1_N -> /ISense2_N
- R13 pad 1: /PWM_Lights1 -> /PWM_Lights2
- R23 pad 2: /CurrentSenseCh2 -> /CurrentSenseCh1
- R29 pad 1: /PWM_Lights2 -> /PWM_Lights1
- R31 pad 1: /ISense1_P -> /ISense2_P
- R31 pad 2: /ISense1_N -> /ISense2_N
- R36 pad 2: /CurrentSenseCh1 -> /CurrentSenseCh2
- R5 pad 1: /ISense2_P -> /ISense1_P
- R5 pad 2: /ISense2_N -> /ISense1_N
- TP1 pad 1: /ISense2_N -> /ISense1_N
- TP10 pad 1: /CurrentSenseCh1 -> /CurrentSenseCh2
- TP2 pad 1: /ISense2_P -> /ISense1_P
- TP3 pad 1: /CurrentSenseCh2 -> /CurrentSenseCh1
- TP5 pad 1: /PWM_Lights2 -> /PWM_Lights1
- TP6 pad 1: /PWM_Lights1 -> /PWM_Lights2
- TP7 pad 1: /ISense1_N -> /ISense2_N
- TP8 pad 1: /ISense1_P -> /ISense2_P
- U1 pad 12: /PWM_Lights2 -> /PWM_Lights1
- U1 pad 3: /ISense2_N -> /ISense1_N
- U1 pad 5: /ISense2_P -> /ISense1_P
- U2 pad 12: /PWM_Lights1 -> /PWM_Lights2
- U2 pad 3: /ISense1_N -> /ISense2_N
- U2 pad 5: /ISense1_P -> /ISense2_P
Routing:
- net /12V_HighPreference: track 0.00 -> 85.4 mm
- net /OpAmpPWR: track 0.00 -> 71.4 mm, vias 0 -> 10
- net /PWM_Lights2: track 0.00 -> 66.3 mm, vias 0 -> 2
- net /ISense1_P: track 0.00 -> 66.3 mm, vias 0 -> 1
- net /ISense2_P: track 0.00 -> 66.3 mm, vias 0 -> 1
- net /ISense1_N: track 0.00 -> 60.7 mm, vias 0 -> 1
- net /ISense2_N: track 0.00 -> 60.5 mm, vias 0 -> 1
- net /ISen2_unfilt: track 0.00 -> 59.8 mm, vias 0 -> 3
- net /PWM_Lights1: track 0.00 -> 47.8 mm
- net Net-(D14-K): track 0.00 -> 47.1 mm
- net /RelaySelectHighPreference: track 0.00 -> 46.4 mm
- net /ISen1_unfilt: track 0.00 -> 45.8 mm, vias 0 -> 1
- net /VIN_OPA_PWR: track 0.00 -> 32.3 mm
- net Net-(Q2-G): track 0.00 -> 28.5 mm
- net /12V_Lights: track 0.00 -> 27.5 mm
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- added copper zone on F.Cu, net /12V_HighPreference
- added copper zone on B.Cu, net /12V_Lights
- added copper zone on F.Cu, net /12V_Lights
- added copper zone on B.Cu, net /12V_LowPreference
- added copper zone on F.Cu, net /12V_LowPreference
- added copper zone on F.Cu, net /ISense1_N
- added copper zone on F.Cu, net /ISense1_P
- added copper zone on F.Cu, net /ISense2_N
- added copper zone on F.Cu, net /ISense2_P
- added copper zone on F.Cu, net /OpAmpPWR
- added copper zone on F.Cu, net /VIN_OPA_PWR
- added copper zone on B.Cu, net GND
- added copper zone on F.Cu, net GND

Commit message: cleaned up routing
Parts:
- added TP11: TestPoint_Small, TestPoint:TestPoint_Pad_D2.0mm, F.Cu at (111.0, 65.0)
- added kibuzzard-65ECAEE6: G***, kibuzzard-65ECAEE6, F.Cu at (154.5, 37.5)
- added kibuzzard-65ECAF22: G***, kibuzzard-65ECAF22, F.Cu at (154.5, 54.5)
- added kibuzzard-65ECAFB8: G***, kibuzzard-65ECAFB8, F.Cu at (138.0, 29.5)
- added kibuzzard-65ECAFEF: G***, kibuzzard-65ECAFEF, F.Cu at (114.5, 29.5)
- added kibuzzard-65ECB040: G***, kibuzzard-65ECB040, F.Cu at (148.5, 62.0)
- added kibuzzard-65ECB075: G***, kibuzzard-65ECB075, F.Cu at (148.5, 89.0)
- added kibuzzard-65ECB164: G***, kibuzzard-65ECB164, F.Cu at (104.5, 62.0)
- added kibuzzard-65ECB19A: G***, kibuzzard-65ECB19A, F.Cu at (125.1, 65.0)
- added kibuzzard-65ECB1C7: G***, kibuzzard-65ECB1C7, F.Cu at (124.0, 69.0)
- added kibuzzard-65ECB1F7: G***, kibuzzard-65ECB1F7, F.Cu at (139.0, 62.0)
- added kibuzzard-65ECB1F7: G***, kibuzzard-65ECB1F7, F.Cu at (155.0, 78.0)
- added kibuzzard-65ECB203: G***, kibuzzard-65ECB203, F.Cu at (155.0, 105.0)
- added kibuzzard-65ECB203: G***, kibuzzard-65ECB203, F.Cu at (139.5, 89.0)
- added kibuzzard-65ECB213: G***, kibuzzard-65ECB213, F.Cu at (124.1, 73.0)
- added kibuzzard-65ECB243: G***, kibuzzard-65ECB243, F.Cu at (123.7, 77.0)
- added kibuzzard-65ECB256: G***, kibuzzard-65ECB256, F.Cu at (123.8, 81.0)
- added kibuzzard-65ECB323: G***, kibuzzard-65ECB323, F.Cu at (181.0, 85.5)
- added kibuzzard-65ECB342: G***, kibuzzard-65ECB342, F.Cu at (181.0, 112.5)
- added kibuzzard-65ECB367: G***, kibuzzard-65ECB367, F.Cu at (108.5, 44.0)
- added kibuzzard-65ECB383: G***, kibuzzard-65ECB383, F.Cu at (133.5, 43.5)
- added kibuzzard-65ECB3CB: G***, kibuzzard-65ECB3CB, F.Cu at (193.0, 62.5)
- added kibuzzard-65ECB3DA: G***, kibuzzard-65ECB3DA, F.Cu at (193.0, 85.5)
- added kibuzzard-65ECB3EB: G***, kibuzzard-65ECB3EB, F.Cu at (193.0, 89.5)
- added kibuzzard-65ECB3F2: G***, kibuzzard-65ECB3F2, F.Cu at (193.0, 112.5)
- added kibuzzard-65ECB486: G***, kibuzzard-65ECB486, F.Cu at (169.0, 85.5)
- added kibuzzard-65ECB57D: G***, kibuzzard-65ECB57D, F.Cu at (161.5, 62.0)
- added kibuzzard-65ECB58F: G***, kibuzzard-65ECB58F, F.Cu at (161.5, 89.0)
- added kibuzzard-65ECB67C: G***, kibuzzard-65ECB67C, F.Cu at (169.0, 112.5)
- added kibuzzard-65ECB6CC: G***, kibuzzard-65ECB6CC, F.Cu at (117.0, 26.0)
- added kibuzzard-65ECB6F2: G***, kibuzzard-65ECB6F2, F.Cu at (176.5, 25.5)
- added kibuzzard-65ECBE96: G***, kibuzzard-65ECBE96, F.Cu at (186.0, 118.0)
- added kibuzzard-65ECDE3F: G***, kibuzzard-65ECDE3F, F.Cu at (174.5, 69.0)
- added kibuzzard-65ECDE69: G***, kibuzzard-65ECDE69, F.Cu at (174.5, 96.0)
- added kibuzzard-65ECDF44: G***, kibuzzard-65ECDF44, F.Cu at (112.0, 92.5)
- added kibuzzard-65ECE287: G***, kibuzzard-65ECE287, F.Cu at (111.9, 94.8)
- J1, J2: footprint TerminalBlock_MetzConnect:TerminalBlock_MetzConnect_Type703_RT10N02HGLU_1x02_P9.52mm_Horizontal -> Connectors_SurgicalLighting:NC6-P108-02
- K1: value Relay_SPDT -> PC792A-1C-C-12S-DN-X
- moved R30 6.11 mm to (169.5, 77.1)
- moved D11 6.06 mm to (169.5, 98.0)
- moved R35 6.02 mm to (169.5, 104.0)
- moved D8 5.93 mm to (169.5, 71.1)
- moved TP4 5.57 mm to (155.0, 84.0)
- moved TP9 5.39 mm to (155.0, 111.0)
- moved J1 3.20 mm to (188.6, 69.3)
- moved J2 3.20 mm to (188.6, 96.2)
- moved TP1 1.80 mm to (173.0, 85.5)
- moved TP2 1.80 mm to (177.0, 85.5)
- moved TP7 1.80 mm to (173.0, 112.5)
- moved TP8 1.80 mm to (177.0, 112.5)
- moved D20 1.50 mm to (177.5, 74.0)
- moved D21 1.48 mm to (177.5, 101.0)
- moved K1 0.95 mm to (173.0, 45.0)
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Connections:
- net Net-(D14-K) renamed /RELAY_COIL_N
- net Net-(Q1-G) renamed /RelayFETGate
- D11 pad 1: /ISense2_P -> Net-(D11-K)
- D11 pad 2: Net-(D11-A) -> /12V_Lights
- D8 pad 1: /ISense1_P -> Net-(D8-K)
- D8 pad 2: Net-(D8-A) -> /12V_Lights
- R30 pad 1: /12V_Lights -> Net-(D8-K)
- R30 pad 2: Net-(D8-A) -> /ISense1_P
- R35 pad 1: /12V_Lights -> Net-(D11-K)
- R35 pad 2: Net-(D11-A) -> /ISense2_P
Routing:
- net /ISense1_N: track 60.7 -> 55.9 mm
- net /ISense1_P: track 66.3 -> 61.5 mm
- net Net-(D11-K): track 0.00 -> 4.15 mm
- net Net-(D11-A): track 4.15 -> 0.00 mm
- net Net-(D8-A): track 4.14 -> 0.00 mm
- net Net-(D8-K): track 0.00 -> 4.13 mm
- net /ISense2_P: track 66.3 -> 62.4 mm
- net /ISense2_N: track 60.5 -> 56.6 mm
- net Net-(Q3-G): track 25.2 -> 26.9 mm
- net Net-(Q2-G): track 28.5 -> 29.9 mm
- net /RELAY_COIL_N: track 47.1 -> 46.6 mm

Commit message: added documentation for troubleshooting
Parts:
- removed kibuzzard-65ECAF22: G***, kibuzzard-65ECAF22
- removed kibuzzard-65ECB367: G***, kibuzzard-65ECB367
- removed kibuzzard-65ECB383: G***, kibuzzard-65ECB383
- added kibuzzard-65F1E0A1: G***, kibuzzard-65F1E0A1, F.Cu at (110.5, 98.7)
- added kibuzzard-65F7788D: G***, kibuzzard-65F7788D, F.Cu at (154.5, 53.7)
- added kibuzzard-65F778BD: G***, kibuzzard-65F778BD, F.Cu at (133.5, 42.7)
- added kibuzzard-65F778C5: G***, kibuzzard-65F778C5, F.Cu at (108.5, 43.2)
- moved R42 2.68 mm to (121.0, 54.7)
- moved C1 0.82 mm to (139.0, 57.2)
- moved C10 0.82 mm to (130.0, 54.2)
- moved C11 0.82 mm to (112.0, 54.2)
- moved C2 0.82 mm to (151.0, 64.2)
- moved C3 0.82 mm to (131.0, 100.1)
- moved C4 0.82 mm to (131.0, 73.2)
- moved C5 0.82 mm to (151.0, 91.2)
- moved C6 0.82 mm to (120.0, 84.2)
- moved C7 0.82 mm to (120.0, 88.2)
- moved C8 0.82 mm to (112.0, 57.2)
- moved C9 0.82 mm to (130.0, 57.2)
- moved D1 0.82 mm to (178.0, 29.2)
- moved D10 0.82 mm to (120.0, 80.2)
- moved D12 0.82 mm to (173.5, 100.2)
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Other:
- board text added: "Troubleshooting (in this order): PWM1/2, RelayEna (if Wall Powered) off -> check for D26-D28 shorts, Replace Logic Board otherwise Gate PWM 1/2 off, PWM1/2 on -> Replace U1/U2 with LM321 RelayEna on, CoilOn off, 12V Wall On -> Check D1,D2 for shorts, otherwise Replace Relay K1, Q1 IRFZ44N 12V to Lights off -> Ensure unit has power from battery / wall, check D3, D20, lights for shorts ICPWRIN on, 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"

Commit message: Moved around stuff
Parts:
- moved J3 0.82 mm to (102.0, 65.4)
